File: SECAM-TDA.sch (EAGLE design)
At the start: 73 parts, among them IC1 MC34063AD

Commit message: .
Parts:
- R7: device rcl:R-EU_R0805 -> rcl:R-EU_0204/7
Changed lines of the file:
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@@
 <part name="GND21" library="supply1" deviceset="GND" device=""/>
 <part name="R5" library="rcl" deviceset="R-EU_" device="0204/7" value="100k"/>
-<part name="R7" library="rcl" deviceset="R-EU_" device="R0805" value="100"/>
+<part name="R7" library="rcl" deviceset="R-EU_" device="0204/7" value="100"/>
 <part name="R8" library="rcl" deviceset="R-EU_" device="R0805" value="22k"/>
 <part name="R10" library="rcl" deviceset="R-EU_" device="R0805" value="1k8"/>
