File: SECAM-TDA.brd (EAGLE design)
At the start: 73 parts, among them IC1 MC34063AD

Commit message: .
Parts:
- R7: device rcl:R0805 -> rcl:0204/7
- moved C11 3.98 mm to (20.3, 25.2), turned to 270 degrees
- moved R7 1.91 mm to (22.5, 28.6), flipped to the top, turned to 0 degrees
Routing:
- net N$9: track 3.55 -> 0.00 mm
- net GND: track 165.3 -> 168.6 mm
- net N$19: track 3.91 -> 2.01 mm
Changed lines of the file:
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@@
 <element name="C9" library="rcl" package="C025-025X050" value="1m" x="19.84375" y="34.13125" rot="R270"/>
 <element name="C10" library="rcl" package="C025-025X050" value="1n" x="24.13" y="33.02" rot="R180"/>
-<element name="C11" library="rcl" package="C025-025X050" value="470n" x="20.0025" y="29.21" rot="R90"/>
+<element name="C11" library="rcl" package="C025-025X050" value="470n" x="20.32" y="25.24125" rot="R270"/>
 <element name="C12" library="rcl" package="C025-025X050" value="6n8" x="24.13" y="30.48" rot="R180"/>
 <element name="C13" library="rcl" package="C025-025X050" value="220n" x="24.13" y="26.51125" rot="R180"/>
@@
 <element name="C26" library="rcl" package="C0805" value="100n" x="60.325" y="56.99125" rot="MR90"/>
 <element name="R5" library="rcl" package="0204/7" value="100k" x="20.32" y="40.9575" rot="R270"/>
-<element name="R7" library="rcl" package="R0805" value="100" x="24.4475" y="28.575" rot="MR180"/>
+<element name="R7" library="rcl" package="0204/7" value="100" x="22.5425" y="28.575"/>
 <element name="R8" library="rcl" package="R0805" value="22k" x="24.13" y="21.9075" rot="MR180"/>
 <element name="R10" library="rcl" package="R0805" value="1k8" x="39.21125" y="25.55875" rot="MR180"/>
@@
 <wire x1="22.86" y1="26.51125" x2="22.86" y2="23.97125" width="0.4064" layer="16"/>
 <wire x1="23.18" y1="21.9075" x2="22.86" y2="23.97125" width="0.4064" layer="16"/>
-<wire x1="22.86" y1="26.51125" x2="18.25625" y2="26.3525" width="0.4064" layer="16"/>
-<wire x1="18.25625" y1="26.3525" x2="18.25625" y2="29.21" width="0.4064" layer="16"/>
-<wire x1="18.25625" y1="29.21" x2="20.0025" y2="30.48" width="0.4064" layer="16"/>
-<wire x1="20.0025" y1="30.48" x2="22.86" y2="30.48" width="0.4064" layer="16"/>
+<wire x1="18.25625" y1="26.3525" x2="18.25625" y2="30.63875" width="0.4064" layer="16"/>
 <wire x1="22.86" y1="33.02" x2="19.84375" y2="32.86125" width="0.4064" layer="16"/>
 <wire x1="27.305" y1="40.005" x2="19.3675" y2="40.005" width="0.4064" layer="16"/>
@@
 <wire x1="30.48" y1="40.48125" x2="30.48" y2="48.5775" width="0.4064" layer="16"/>
 <wire x1="30.48" y1="48.5775" x2="30.3865125" y2="51.276975" width="0.4064" layer="16"/>
+<wire x1="22.86" y1="30.48" x2="18.25625" y2="30.63875" width="0.4064" layer="16"/>
+<wire x1="20.32" y1="23.97125" x2="18.415" y2="23.97125" width="0.4064" layer="16"/>
+<wire x1="18.415" y1="23.97125" x2="18.25625" y2="26.3525" width="0.4064" layer="16"/>
 <wire x1="111.76" y1="30.89625" x2="114.3" y2="30.89625" width="0" layer="19" extent="1-1"/>
 <wire x1="98.425" y1="17.30375" x2="111.76" y2="30.89625" width="0" layer="19" extent="1-1"/>
@@
 <wire x1="41.43125" y1="39.52875" x2="41.91" y2="47.14875" width="0" layer="19" extent="16-16"/>
 <wire x1="43.4975" y1="39.37" x2="41.43125" y2="39.52875" width="0" layer="19" extent="16-16"/>
-<wire x1="46.99" y1="28.895" x2="43.4975" y2="39.37" width="0" layer="19" extent="16-16"/>
+<wire x1="46.99" y1="28.895" x2="55.2425" y2="35.2425" width="0" layer="19" extent="16-16"/>
 <wire x1="42.06875" y1="28.41625" x2="46.99" y2="28.895" width="0" layer="19" extent="16-16"/>
+<wire x1="20.32" y1="23.97125" x2="22.86" y2="23.97125" width="0.4064" layer="16"/>
 </signal>
 <signal name="N$2">
@@
 <contactref element="R7" pad="2"/>
 <wire x1="27.305" y1="31.115" x2="25.4" y2="30.48" width="0.4064" layer="16"/>
-<wire x1="25.4" y1="30.48" x2="25.3975" y2="28.575" width="0.4064" layer="16"/>
+<wire x1="25.4" y1="30.48" x2="26.3525" y2="28.575" width="0" layer="19" extent="1-16"/>
 </signal>
 <signal name="N$9">
 <contactref element="C11" pad="1"/>
 <contactref element="R7" pad="1"/>
-<wire x1="23.4975" y1="28.575" x2="20.0025" y2="27.94" width="0.4064" layer="16"/>
+<wire x1="18.7325" y1="28.575" x2="20.32" y2="26.51125" width="0" layer="19" extent="1-16"/>
 </signal>
 <signal name="N$18">

Commit message: .
Parts:
- removed 1R1: 27K, resistor:R0805
- removed 2L2: 220uH, inductor-neosid:SD12_1000
- added 3VD2: SS12, diode:SMB
- added C27: 36, rcl:C0805
- added C28: 100n, rc-elektronik:C0805
- added C29: 1n, rcl:C0805
- added C30: 470µ, HWProgUSB:RCL_E2,5-7
- added C35, C36: 100n, rcl:C0805
- added C37, C38: 100µ 16V, HWProgUSB:RCL_E2,5-5
- added DA4: MC34063AD, mc34063:SOIC8
- added DA5: 78L06, ct-pack:SOT89R
- added IC2: (no value), ic-package:DIL40
- added JP1, JP2, JP3: (no value), Разъёмы штырьковые 2.54мм:1X20
- added JP4: (no value), jumper:JP1
- added L2: (no value), rcl:0204/5
- added L2.2: (no value), pinhead:1X01
- added L3, L4: (no value), rcl:0204/7
- added L5: 100uh, rcl:0204/7
- added L6: 100uh, rcl:0207/10
- added R28: 4k7, rcl:R0805
- added R29: 180, rcl:M0805
- added R30: 0.5, rcl:M1206
- added R31: 7k5(9k1 6v), rcl:M0805
- added R32: 1k5(2k4 6v), rcl:M0805
- added S1: (no value), ESR_NM8032:SWITCH9X4
- added SJ1: (no value), jumper:SJ
- added U$5: B-, ESR_NM8032:B-
- added U$6: B+, ESR_NM8032:B+
- 2D2: device diode:DO41-10 -> diode:SMB
- C33: value 100n -> 100µ 16V; device resistor:C0805K -> HWProgUSB:RCL_E2,5-5
- moved C33 179.9 mm to (-5.08, -121.9)
Connections:
- new net +6V: C28.1, C30.+, DA4.6, R30.1, U$6.P$1
- new net N$47: C27.1, JP4.1, R28.2
- new net N$48: R1.3, R2.3, R3.3, SJ1.1
- new net N$49: DA1.22, JP4.2, R28.1
- new net N$58: C27.2, L2.2
- new net N$59: DA4.7, L5.1, R29.2, R30.2
- new net N$60: DA4.5, R31.1, R32.2
- new net N$61: 3VD2.A, DA4.1, L5.2
- new net N$62: C29.1, DA4.3
- new net N$63: 3VD2.C, C33.+, C35.2, L6.1, R31.2
- new net N$64: S1.12, S1.22, U$5.P$1
- new net N$65: S1.11, S1.21
- new net N$66: C36.1, C37.+, DA5.1, L6.2
- new net V+: C38.+, DA5.2
- net +5V: now also L3.2
- net GND: now also C1.2, C28.2, C29.2, C30.-, C33.-, C35.1, C36.2, C37.-, C38.-, DA4.2, DA4.4, DA5.3, DA5.4, L2.1, R32.1, S1.10, S1.20; no longer C1.1, R1.3, R2.3, R3.3
- net N$51: now also L4.2; no longer 2L2.2
- net N$52: now also L4.1; no longer 2L2.1
- net N$55: now also DA4.8, L2.2.1, R29.1; no longer 1R1.2, C33.1
- net N$56: no longer 1R1.1
- net N$57: now also L3.1
- net N$6: now also C1.1, SJ1.2; no longer C1.2
Routing:
- net GND: track 168.6 -> 150.4 mm
